File: entradas.kicad_sch (KiCad schematic)
At the start: 16 parts, among them J4 entrada discreta, J5 entrada discreta, SW1 SW_MEC_5E, SW2 SW_MEC_5E, U4 LTV-817-C, U5 LTV-817-C

Commit message: organização e legendas do esquemático
Other:
- moved on the sheet: D2, D3, J4, J5, R10, R11, R12, R13, R14, R15, R16, R9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

Commit message: ajusta circuitos de entrada, alimentação e saída e adiciona visualizações da PCB
Parts:
- removed R11, R12, R13, R14: 0603WAF1001T5E, jlclib:R0603, symbol a_jlclib:0603WAF1001T5E
- added R11, R12, R13, R14: 0805W8F1001T5E, jlclib:R0805, symbol a_jlclib:0805W8F1001T5E
Connections:
- net 3V3_IN: now also U4.4, U5.4; no longer R15.2, R16.2
- net ED1: now also R15.2, U4.3; no longer R15.1, U4.4
- net ED2: now also R16.2, U5.3; no longer R16.1, U5.4
- net GND: now also R15.1, R16.1, R12.1, R14.1; no longer U4.3, U5.3
- net at U4.2: now also R11.2
- net at U5.2: now also R13.2
- new net: R13.1, R14.2
- new net: R11.1, R12.2
Other:
- moved on the sheet: R15, R16
