File: pcb-moduloDidaticoSCADA.kicad_pcb (KiCad board)
At the start: 2 copper layers, 100 x 100 mm, 92 parts, among them J1 alimentação 12 Vcc, J10 CARGA_12V, J11 JUMP 120R, J12 Habilita buzzer, J13 Habilita rele, J2 RS485, J3 DS18B20, J4 entrada discreta, J5 entrada discreta, J6 MOTOR, J7 PWM_SERVO, J8 PWM_SERVO, J9 Screw_Terminal_01x03, K1 Relay_SPDT_Latching_1coil, Q1 2N7002, Q2 SI4483ADY-T1-GE3, Q3 2N7002, Q4 2N7002, SW1 SW_MEC_5E, SW2 SW_MEC_5E, U1 NODEMCU, U2 LM317G, U3 AMS1117-5.0, U4 LTV-817-C, U5 LTV-817-C, U6 AS4950, U7 SP3485EN-L/TR_C41365340

Commit message: style: ajustes no layout
Parts:
- removed REF**: KiCad-Logo2_5mm_SilkScreen, Symbol:KiCad-Logo2_5mm_SilkScreen
- removed REF**: Screw_Generic_2.0x3.0mm_SilkScreen, Symbol:Screw_Generic_2.0x3.0mm_SilkScreen
- added D12: LED, LED_THT:LED_D5.0mm, F.Cu at (68.0, 93.0)
- added R36: 0603WAF1201T5E, jlclib:R0603, F.Cu at (67.5, 98.0)
- RV1: value R_Potentiometer_Trim -> 20K
Connections:
- net /PWM_LAMP/D1/IO5 renamed /PWM_RESISTENCIA/D1/IO5
- RV1 pad 3: /EA1/A0/ADC -> /3V3

Commit message: ajustes no layout e serigrafia
Parts:
- removed D12: LED, LED_THT:LED_D5.0mm
- removed D7: SS12 Schottky, Diode_SMD:D_SMA_Handsoldering
- removed J10: CARGA_12V, Connector_PinSocket_2.54mm:PinSocket_1x02_P2.54mm_Vertical
- removed R36: 0603WAF1201T5E, jlclib:R0603
- added C12: 10uFx50V, Capacitor_THT:CP_Radial_D5.0mm_P2.50mm, F.Cu at (187.2, 127.8)
- added G***: LOGO, imagens:qrfirmware, B.Cu at (172.3, 65.9)
- added G***: LOGO, imagens:qrpcb, B.Cu at (172.4, 90.9)
- added H5: MountingHole, MountingHole:MountingHole_3.2mm_M3, F.Cu at (159.7, 61.7)
- added H6: MountingHole, MountingHole:MountingHole_3.2mm_M3, F.Cu at (186.4, 61.7)
- added H7: MountingHole, MountingHole:MountingHole_3.2mm_M3, F.Cu at (159.7, 92.7)
- added H8: MountingHole, MountingHole:MountingHole_3.2mm_M3, F.Cu at (186.4, 92.7)
- added R37: 15R10W, Resistor_THT:R_Axial_Power_L38.0mm_W9.0mm_P40.64mm, F.Cu at (98.0, 134.8)
- added REF**: KiCad-Logo2_6mm_SilkScreen, Symbol:KiCad-Logo2_6mm_SilkScreen, F.Cu at (146.3, 118.4)
- added REF**: KiCad-Logo2_5mm_SilkScreen, Symbol:KiCad-Logo2_5mm_SilkScreen, F.Cu at (105.5, 145.5)
- added REF**: KiCad-Logo2_12mm_SilkScreen, Symbol:KiCad-Logo2_12mm_SilkScreen, B.Cu at (143.6, 120.0)
- added U8: AMS1117-5.0, jlclib:SOT-223_L6.5-W3.5-P2.30-LS7.0-BR, F.Cu at (186.4, 121.6)
- J6: footprint Connector_PinSocket_2.54mm:PinSocket_1x02_P2.54mm_Vertical -> TerminalBlock:TerminalBlock_MaiXu_MX126-5.0-02P_1x02_P5.00mm
- moved R20 25.3 mm to (113.5, 123.8)
- moved R19 24.9 mm to (116.9, 123.8), turned to 180 degrees
- moved Q1 23.2 mm to (116.6, 120.9), turned to 0 degrees
- moved J3 19.9 mm to (104.6, 103.6), turned to 0 degrees
- moved R22 18.6 mm to (113.9, 119.0), turned to 90 degrees
- moved R23 14.9 mm to (111.8, 118.9), turned to -90 degrees
- moved R25 14.0 mm to (112.0, 112.4), turned to 90 degrees
- moved R4 13.3 mm to (107.6, 107.9), turned to 90 degrees
- moved D8 12.3 mm to (109.0, 113.7), turned to 180 degrees
- moved Q2 11.7 mm to (107.1, 120.1), turned to 90 degrees
- moved D4 11.6 mm to (118.2, 59.1)
- moved R17 11.6 mm to (121.5, 59.3)
- moved J12 11.6 mm to (125.1, 59.1)
- moved Q4 10.9 mm to (114.2, 53.6)
- moved R34 10.8 mm to (119.2, 53.7), turned to 90 degrees
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Connections:
- C10 pad 1: +5V -> +5V_SERVO
- C11 pad 1: +5V -> +5V_SERVO
- C8 pad 2: +5V -> /3V3
- D10 pad 2: /PWM_AZ/D7/IO13 -> /PWM_EL/D3/IO0
- D9 pad 2: /PWM_EL/D3/IO0 -> /PWM_AZ/D7/IO13
- J3 pad 3: /3.3V -> /3V3
- J7 pad 2: +5V -> +5V_SERVO
- J7 pad 3: /PWM_EL/D3/IO0 -> /PWM_AZ/D7/IO13
- J8 pad 2: +5V -> +5V_SERVO
- J8 pad 3: /PWM_AZ/D7/IO13 -> /PWM_EL/D3/IO0
- R4 pad 1: /3.3V -> /3V3
- U1 pad 1: /RST -> unconnected-(U1-RST-Pad1)
- U1 pad 13: /RST -> unconnected-(U1-RST-Pad13)
- U1 pad 16: /3.3V -> /3V3
- U6 pad 6: Net-(J6-Pin_1) -> Net-(J6-Pin_2)
- U6 pad 8: Net-(J6-Pin_2) -> Net-(J6-Pin_1)
Routing:
- net +12V: track 59.2 -> 244.0 mm
- net /SD2/TXD0/GPIO1: track 4.34 -> 154.6 mm
- net /3V3: track 0.00 -> 141.6 mm, vias 0 -> 2
- net +5V: track 46.4 -> 166.8 mm, vias 3 -> 4
- net 7V5: track 1.98 -> 101.7 mm, vias 0 -> 12
- net /SD1/D0/IO16: track 5.89 -> 95.5 mm
- net /PWM_RESISTENCIA/D1/IO5: track 0.00 -> 72.4 mm
- net /ED2/RXD0/GPIO3: track 0.00 -> 67.9 mm, vias 0 -> 1
- net /DATA_DS18B20/IO4: track 0.00 -> 61.2 mm, vias 0 -> 2
- net /ED1/D8/IO15-config: track 0.27 -> 50.2 mm, vias 0 -> 2
- net /PWM_AZ/D7/IO13: track 6.10 -> 43.4 mm
- net +5V_SERVO: track 0.00 -> 27.7 mm
- net /PWM_EL/D3/IO0: track 6.07 -> 32.8 mm
- net Net-(D8-A): track 3.81 -> 24.6 mm
- net Net-(D6-A): track 0.00 -> 20.6 mm
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- added copper zone on F.Cu, net +5V_SERVO
- added copper zone on F.Cu, net /3V3
- added copper zone on B.Cu, net 7V5
Other:
- outline, holes or cut-outs redrawn
- board text added: "07/2026"
- board text added: "BY WILLIAM"
- board text added: "FIRMWARE"
- board text added: "GND 5V S"
- board text added: "PROJETO PCB"
- board text added: "SERVO MOTORES"
- board text removed: "Config."
- board text removed: "EA1"
- board text removed: "ED1 (SETUP)"
- board text removed: "ED2"
- board text removed: "SD1 - PWM"
- board text removed: "SD2"
- board text removed: "SD2 - PWM"
- board text removed: "SD3 - PWM RESITÊNCIA"
- board text removed: "TEMPERATURA (DS18B20)"
- board text removed: "WEB SERVER MODO SETUP AP (ACCESS POINT) 192.168.4.1"

Commit message: ajusta circuitos de entrada, alimentação e saída e adiciona visualizações da PCB
Parts:
- removed REF**: KiCad-Logo2_6mm_SilkScreen, Symbol:KiCad-Logo2_6mm_SilkScreen
- removed REF**: KiCad-Logo2_5mm_SilkScreen, Symbol:KiCad-Logo2_5mm_SilkScreen
- removed REF**: KiCad-Logo2_12mm_SilkScreen, Symbol:KiCad-Logo2_12mm_SilkScreen
- added R36: 43K, Resistor_SMD:R_0805_2012Metric_Pad1.20x1.40mm_HandSolder, F.Cu at (137.9, 97.2)
- R1, R11, R12, R13, R14, R17, R18, R2, R3, R8: value 0603WAF1001T5E -> 0805W8F1001T5E; footprint jlclib:R0603 -> jlclib:R0805
- moved R6 6.23 mm to (104.8, 133.4), turned to 90 degrees
- moved R24 5.85 mm to (130.5, 95.5), turned to 90 degrees
- moved R7 4.19 mm to (106.8, 133.4), turned to -90 degrees
- moved R5 3.49 mm to (106.0, 129.1)
- moved R20 1.59 mm to (112.8, 122.4), turned to 90 degrees
- moved U6 1.45 mm to (108.0, 68.6)
- moved R18 1.25 mm to (119.7, 70.7)
- moved R28 1.16 mm to (169.5, 123.3)
- moved R16 1.04 mm to (142.0, 91.9)
- moved G*** 0.95 mm to (173.1, 65.5)
- moved R3 0.86 mm to (172.8, 122.9)
- moved D5 0.81 mm to (116.5, 70.3)
- moved R19 0.80 mm to (116.1, 123.9)
- moved R15 0.75 mm to (153.7, 92.0)
- moved J6 0.72 mm to (99.8, 70.8)
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Connections:
- R15 pad 1: /ED1/D8/IO15-config -> GND
- R15 pad 2: /3V3 -> /ED1/D8/IO15-config
- R16 pad 1: /ED2/RXD0/GPIO3 -> GND
- R16 pad 2: /3V3 -> /ED2/RXD0/GPIO3
- RV1 pad 3: /3V3 -> Net-(R36-Pad2)
- U4 pad 3: GND -> /ED1/D8/IO15-config
- U4 pad 4: /ED1/D8/IO15-config -> /3V3
- U5 pad 3: GND -> /ED2/RXD0/GPIO3
- U5 pad 4: /ED2/RXD0/GPIO3 -> /3V3
Routing:
- net Net-(R36-Pad2): track 0.00 -> 18.2 mm
- net /3V3: track 141.6 -> 134.1 mm
- net /ED1/D8/IO15-config: track 50.2 -> 46.5 mm
- net /ED2/RXD0/GPIO3: track 67.9 -> 64.4 mm, vias 1 -> 2
- net /SD2/TXD0/GPIO1: track 154.6 -> 157.8 mm
- net Net-(U2-ADJ): track 7.58 -> 4.54 mm
- net 7V5: track 101.7 -> 104.3 mm
- net Net-(Q3-G): track 8.29 -> 10.6 mm
- net Net-(R5-Pad1): track 1.80 -> 3.83 mm
- net Net-(Q1-G): track 4.47 -> 6.08 mm
- net +12V: track 244.0 -> 245.1 mm
- net Net-(R2-Pad1): track 5.78 -> 6.81 mm
- net /PWM_RESISTENCIA/D1/IO5: track 72.4 -> 73.4 mm
- net Net-(R13-Pad2): track 2.54 -> 3.51 mm
- net Net-(R11-Pad2): track 2.75 -> 3.64 mm
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Other:
- outline, holes or cut-outs redrawn
- board text added: "ANALÓGICA"
- board text added: "ENTRADAS DISCRETAS LOG NOT"
- board text added: "FONTE"
- board text added: "MANUAL DO PROJETO"
- board text added: "NODEMCU"
- board text added: "PCB MÓDULO DIDÁTICO"
- board text added: "RS 485"
- board text added: "SAÍDAS DISCRETAS"
- board text added: "SAÍDAS PWM"
- board text added: "SENSOR ATUADOR"
- board text removed: "LOG INVERTIDA"
